File: ATesp32.kicad_pcb (KiCad board)
At the start: 4 copper layers, 18 x 51.2 mm, 51 parts, among them J1 USB_C_Receptacle_USB2.0_16P, J2 JST PH, Q1 DMP2045U, SW1 RESET, SW2 BOOT, U1 ESP32-S3, U2 ATmega32A-P, U3 MCP73831-2-OT, U4 AP2112K-3.3, U5 CP2102N-Axx-xQFN24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

Commit message: small layout optimization
Parts:
- moved C7 1.20 mm to (83.6, 73.7)
Routing:
- net GND: track 12.0 -> 11.4 mm, vias 108 -> 113
Changed lines of the file:
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@@
 	(footprint "Capacitor_SMD:C_0402_1005Metric"
 		(layer "F.Cu")
-		(at 84.5 74.5 135)
+		(at 83.6 73.7 135)
 		(descr "Capacitor SMD 0402 (1005 Metric), square (rectangular) end terminal, IPC_7351 nominal, (Body size source: IPC-SM-782 page 76, https://www.pcb-3d.com/wordpress/wp-content/uploads/ipc-sm-782a_amendment_1_and_2.pdf), generated with kicad-footprint-generator")
 		(tags "capacitor")
@@
 	)
 	(segment
-		(start 84.160589 74.160589)
-		(end 83.7 73.7)
-		(width 0.5)
-		(layer "F.Cu")
-		(net 3)
-	)
-	(segment
 		(start 79.021178 74.4)
 		(end 79.360589 74.739411)
@@
 	)
 	(via
+		(at 88.5 60.25)
+		(size 0.3)
+		(drill 0.2)
+		(layers "F.Cu" "B.Cu")
+		(free yes)
+		(net 3)
+	)
+	(via
+		(at 87.8 60.5)
+		(size 0.3)
+		(drill 0.2)
+		(layers "F.Cu" "B.Cu")
+		(net 3)
+	)
+	(via
 		(at 82.5 69.75)
 		(size 0.3)
@@
 	)
 	(via
-		(at 87.8 60.5)
-		(size 0.6)
-		(drill 0.3)
+		(at 79 58)
+		(size 0.3)
+		(drill 0.2)
 		(layers "F.Cu" "B.Cu")
+		(free yes)
 		(net 3)
 	)
 	(via
-		(at 79 58)
+		(at 89.5 59.75)
 		(size 0.3)
 		(drill 0.2)
@@
 	)
 	(via
+		(at 89.5 60.25)
+		(size 0.3)
+		(drill 0.2)
+		(layers "F.Cu" "B.Cu")
+		(free yes)
+		(net 3)
+	)
+	(via
 		(at 79.75 59.5)
 		(size 0.3)
@@
 	)
 	(via
+		(at 88.5 59.75)
+		(size 0.3)
+		(drill 0.2)
+		(layers "F.Cu" "B.Cu")
+		(free yes)
+		(net 3)
+	)
+	(via
 		(at 81.74 92.51)
 		(size 0.3)
@@
 	)
 	(via
+		(at 83.798959 72.798958)
+		(size 0.3)
+		(drill 0.2)
+		(layers "F.Cu" "B.Cu")
+		(free yes)
+		(net 3)
+	)
+	(via
 		(at 87.75 76.5)
 		(size 0.3)
@@
 	)
 	(via
+		(at 89 59.75)
+		(size 0.3)
+		(drill 0.2)
+		(layers "F.Cu" "B.Cu")
+		(free yes)
+		(net 3)
+	)
+	(via
 		(at 82.5 59.75)
 		(size 0.3)
@@
 	)
 	(via
-		(at 83.7 73.7)
-		(size 0.6)
-		(drill 0.3)
-		(layers "F.Cu" "B.Cu")
-		(net 3)
-	)
-	(via
 		(at 78.75 56)
 		(size 0.3)
@@
 	)
 	(via
+		(at 89 60.25)
+		(size 0.3)
+		(drill 0.2)
+		(layers "F.Cu" "B.Cu")
+		(free yes)
+		(net 3)
+	)
+	(via
 		(at 83.259699 92.741807)
 		(size 0.3)
@@
 	)
 	(via
-		(at 85.75 70.75)
-		(size 0.3)
-		(drill 0.2)
-		(layers "F.Cu" "B.Cu")
-		(free yes)
-		(net 3)
-	)
-	(via
 		(at 82.5 62.25)
 		(size 0.3)
@@
 	)
 	(segment
-		(start 84.9 74.049098)
-		(end 84.9 62.586827)
+		(start 78.568844 79.031156)
+		(end 79.917942 79.031156)
 		(width 0.15)
 		(layer "B.Cu")
@@
 	)
 	(segment
-		(start 79.917942 79.031156)
-		(end 84.9 74.049098)
+		(start 85.4 62.086827)
+		(end 91.036827 56.45)
 		(width 0.15)
 		(layer "B.Cu")
@@
 	)
 	(segment
-		(start 78.568844 79.031156)
-		(end 79.917942 79.031156)
+		(start 85.4 73.549098)
+		(end 85.4 62.086827)
 		(width 0.15)
 		(layer "B.Cu")
@@
 	)
 	(segment
-		(start 84.9 62.586827)
-		(end 91.036827 56.45)
+		(start 79.917942 79.031156)
+		(end 85.4 73.549098)
 		(width 0.15)
 		(layer "B.Cu")
@@
 	)
 	(segment
-		(start 84.5 73.954124)
-		(end 84.5 61.03)
+		(start 85.05 73.404124)
+		(end 85.05 60.48)
 		(width 0.15)
 		(layer "B.Cu")
@@
 	)
 	(segment
-		(start 79.921987 78.532137)
-		(end 84.5 73.954124)
+		(start 85.05 60.48)
+		(end 91.62 53.91)
 		(width 0.15)
 		(layer "B.Cu")
@@
 	)
 	(segment
-		(start 84.5 61.03)
-		(end 91.62 53.91)
+		(start 78.600156 78.532137)
+		(end 79.921987 78.532137)
 		(width 0.15)
 		(layer "B.Cu")
@@
 	)
 	(segment
-		(start 78.600156 78.532137)
-		(end 79.921987 78.532137)
+		(start 79.921987 78.532137)
+		(end 85.05 73.404124)
 		(width 0.15)
 		(layer "B.Cu")
@@
 	)
 	(segment
-		(start 83 59.99)
-		(end 83 74.198959)
+		(start 84.7 58.29)
+		(end 84.7 72.498959)
 		(width 0.15)
 		(layer "B.Cu")
@@
 	)
 	(segment
-		(start 91.62 51.37)
-		(end 83 59.99)
+		(start 84.7 72.498959)
+		(end 79.183489 78.01547)
 		(width 0.15)
 		(layer "B.Cu")
@@
 	)
 	(segment
-		(start 83 74.198959)
-		(end 79.183489 78.01547)
+		(start 91.62 51.37)
+		(end 84.7 58.29)
 		(width 0.15)
 		(layer "B.Cu")
@@
 	)
 	(segment
-		(start 85.25 65.36)
-		(end 91.62 58.99)
+		(start 85.75 73.694072)
+		(end 85.75 64.86)
 		(width 0.15)
 		(layer "B.Cu")
@@
 	)
 	(segment
-		(start 85.25 74.194072)
-		(end 85.25 65.36)
+		(start 79.672557 79.771515)
+		(end 85.75 73.694072)
 		(width 0.15)
 		(layer "B.Cu")
@@
 	)
 	(segment
-		(start 79.672557 79.771515)
-		(end 85.25 74.194072)
+		(start 85.75 64.86)
+		(end 91.62 58.99)
 		(width 0.15)
 		(layer "B.Cu")
@@
 			)
 		)
+	)
+	(zone
+		(net 3)
+		(net_name "GND")
+		(layer "F.Cu")
+		(hatch edge 0.5)
+		(priority 20)
+		(connect_pads thru_hole_only
+			(clearance 0)
+		)
+		(min_thickness 0.25)
+		(filled_areas_thickness no)
+		(fill yes
+			(thermal_gap 0.5)
+			(thermal_bridge_width 0.5)
+		)
+		(polygon
+			(pts
+				(xy 87.5 61.25) (xy 87.5 60.4) (xy 88.4 59.5) (xy 89.75 59.5) (xy 89.75 61.25)
+			)
+		)
