File: ATesp32_POWER.kicad_sch (KiCad schematic)
At the start: 12 parts, among them J2 JST PH, Q1 DMP2045U, U3 MCP73832-2, U4 AP2112K-3.3

Commit message: generated manf files. Too damn expensive, adjusting min track and holes
Parts:
- C13, C14: JLC C315248 -> (none); LCSC (none) -> C315248
- D2: JLC C510300 -> (none); LCSC (none) -> C510300
- D4: JLC C48192 -> (none); LCSC (none) -> C48192
- J2: JLC C295747 -> (none); LCSC (none) -> C295747
- Q1: JLC C459541 -> (none); LCSC (none) -> C459541
- R2, R4: JLC C25741 -> (none); LCSC (none) -> C25741
- R3: JLC C25744 -> (none); LCSC (none) -> C25744
- R6: JLC C25905 -> (none); LCSC (none) -> C25905
- U3: JLC C38066 -> (none); LCSC (none) -> C38066
- U4: JLC C51118 -> (none); LCSC (none) -> C51118
Changed lines of the file:
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@@
 			)
 		)
-		(property "JLC" "C510300"
+		(property "LCSC" "C510300"
 			(at 113.03 149.86 0)
 			(effects
@@
 			)
 		)
-		(property "JLC" "C315248"
-			(at 97.79 83.82 0)
-			(effects
-				(font
-					(size 1.27 1.27)
-				)
-				(hide yes)
-			)
-		)
 		(property "Sim.Device" ""
 			(at 97.79 83.82 0)
@@
 			)
 		)
+		(property "LCSC" "C315248"
+			(at 97.79 83.82 0)
+			(effects
+				(font
+					(size 1.27 1.27)
+				)
+				(hide yes)
+			)
+		)
 		(pin "1"
 		)
@@
 			)
 		)
-		(property "JLC" "C51118"
+		(property "LCSC" "C51118"
 			(at 118.11 73.66 0)
 			(effects
@@
 			)
 		)
-		(property "JLC" "C315248"
-			(at 109.22 128.27 0)
-			(effects
-				(font
-					(size 1.27 1.27)
-				)
-				(hide yes)
-			)
-		)
 		(property "Sim.Device" ""
 			(at 109.22 128.27 0)
@@
 			)
 		)
+		(property "LCSC" "C315248"
+			(at 109.22 128.27 0)
+			(effects
+				(font
+					(size 1.27 1.27)
+				)
+				(hide yes)
+			)
+		)
 		(pin "1"
 		)
@@
 			)
 		)
-		(property "JLC" "C25905"
+		(property "LCSC" "C25905"
 			(at 99.06 144.78 0)
 			(effects
@@
 			)
 		)
-		(property "JLC" "C38066"
+		(property "LCSC" "C38066"
 			(at 88.9 124.46 0)
 			(effects
@@
 			)
 		)
-		(property "JLC" "C25744"
+		(property "LCSC" "C25744"
 			(at 74.93 132.08 0)
 			(effects
@@
 			)
 		)
-		(property "JLC" "C459541"
+		(property "LCSC" "C459541"
 			(at 92.71 54.61 0)
 			(effects
@@
 			)
 		)
-		(property "JLC" "C25741"
+		(property "LCSC" "C25741"
 			(at 100.33 74.93 0)
 			(effects
@@
 			)
 		)
-		(property "JLC" "C25741"
+		(property "LCSC" "C25741"
 			(at 82.55 78.74 0)
 			(effects
@@
 			)
 		)
-		(property "JLC" "C295747"
+		(property "LCSC" "C295747"
 			(at 127 121.92 0)
 			(effects
@@
 			)
 		)
-		(property "JLC" "C48192"
+		(property "LCSC" "C48192"
 			(at 87.63 71.12 0)
 			(effects

Commit message: Add some Mouser PNs
Parts:
- C13, C14: DigiKey (none) -> 1276-1450-1-ND
- D2: DigiKey (none) -> SML-P11UTT86RCT-ND
- D4: DigiKey (none) -> NSR0320MW2T1GOSCT-ND
Changed lines of the file:
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@@
+			)
+		)
+		(property "DigiKey" "SML-P11UTT86RCT-ND"
+			(at 113.03 149.86 0)
+			(effects
+				(font
+					(size 1.27 1.27)
+				)
+				(hide yes)
 			)
 		)
@@
 			)
 		)
+		(property "DigiKey" "1276-1450-1-ND"
+			(at 97.79 83.82 0)
+			(effects
+				(font
+					(size 1.27 1.27)
+				)
+				(hide yes)
+			)
+		)
 		(pin "1"
 		)
@@
 			)
 		)
+		(property "DigiKey" "1276-1450-1-ND"
+			(at 109.22 128.27 0)
+			(effects
+				(font
+					(size 1.27 1.27)
+				)
+				(hide yes)
+			)
+		)
 		(pin "1"
 		)
@@
 			(at 87.63 71.12 0)
 			(effects
+				(font
+					(size 1.27 1.27)
+				)
+				(hide yes)
+			)
+		)
+		(property "DigiKey" "NSR0320MW2T1GOSCT-ND"
+			(at 87.63 71.12 0)
+			(effects

Commit message: update manf outputs
Parts:
- U3: value MCP73832-2 -> MCP73832T-2; DigiKey (none) -> MCP73832T-2ACI/OTCT-ND
- U4: DigiKey (none) -> AP2112K-3.3TRG1DICT-ND
Changed lines of the file:
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@@
+			)
+		)
+		(property "DigiKey" "AP2112K-3.3TRG1DICT-ND"
+			(at 118.11 73.66 0)
+			(effects
+				(font
+					(size 1.27 1.27)
+				)
+				(hide yes)
 			)
 		)
@@
 			)
 		)
-		(property "Value" "MCP73832-2"
+		(property "Value" "MCP73832T-2"
 			(at 91.0941 116.84 0)
 			(effects
@@
 			(at 88.9 124.46 0)
 			(effects
+				(font
+					(size 1.27 1.27)
+				)
+				(hide yes)
+			)
+		)
+		(property "DigiKey" "MCP73832T-2ACI/OTCT-ND"
+			(at 88.9 124.46 0)
+			(effects
